Commit message: Update 07_pantilt.urdf

File: urdf/07_pantilt.urdf (robot description, URDF)
Before this commit: robot pan_tilt, 4 links, 3 joints
Links:
- link base_link: geometry visual mesh filename=package://pantilt_ros/meshes/baza.STL
- link pan_link: geometry visual mesh filename=package://pantilt_ros/meshes/pan_stalp.STL
