Commit message: Update 08_pantilt.urdf

File: urdf/08_pantilt.urdf (robot description, URDF)
Before this commit: robot pan_tilt, 4 links, 3 joints
Links:
- link base_link: geometry visual mesh filename=package://pantilt_ros/meshes/baza.STL
- link pan_link: geometry visual mesh filename=package://robotel/pantilt_ros/pan_stalp.STL
- link tilt_link: geometry visual mesh filename=package://pantilt_ros/meshes/tilt_stalp.STL

Commit message: Update 08_pantilt.urdf

File: urdf/08_pantilt.urdf (robot description, URDF)
Before this commit: robot pan_tilt, 4 links, 3 joints
Links:
- link pan_link: geometry visual mesh filename=package://pantilt_ros/pan_stalp.STL

Commit message: Update 08_pantilt.urdf

File: urdf/08_pantilt.urdf (robot description, URDF)
Before this commit: robot pan_tilt, 4 links, 3 joints
Links:
- link pan_link: geometry visual mesh filename=package://pantilt_ros/meshes/pan_stalp.STL
